File: clock.kicad_sch (KiCad schematic)
At the start: 5 parts, among them U36 NE555P

Commit message: very big comit what i did is in the description
jooo so this is what i did i fixed all erc errors now it is basicly finished and also started to make a website where you can lern how this whole thing works and also have a simulation for it but it is still in progress so right now chapter 1 is complete with all the simulations and right now i am working on chapter 6 it should not take very long untill i am finished i will probaply post more comits in the future so yea sry that i forgot to do that ig
Parts:
- U36: value NE555P -> TLC555
Changed lines of the file:
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@@
 			)
 		)
-		(property "Value" "NE555P"
+		(property "Value" "TLC555"
 			(at 57.15 35.4898 0)
 			(show_name no)
