File: counter.kicad_sch (KiCad schematic)
At the start: 14 parts, among them U1 74HC192, U2 74HC192, U4 74AHC1G08, U5 74AHC1G08, U68 74AHC1G32, U69 74AHC1G32, U70 74AHC1G02, U71 74AHC1G02, U72 74AHC1G02, U73 74AHC1G02, U74 74AHC1G02, U75 74AHC1G02, U8 74AHC1G08, U9 74AHC1G08

Commit message: very big comit what i did is in the description
jooo so this is what i did i fixed all erc errors now it is basicly finished and also started to make a website where you can lern how this whole thing works and also have a simulation for it but it is still in progress so right now chapter 1 is complete with all the simulations and right now i am working on chapter 6 it should not take very long untill i am finished i will probaply post more comits in the future so yea sry that i forgot to do that ig
Parts:
- added U3: 74AHC1G32, symbol 74xGxx:74AHC1G32
Connections:
- net +3V3: now also U73.5 (VCC), U74.5 (VCC), U3.5 (VCC)
- net GND: now also U73.3 (GND), U74.3 (GND), U3.3 (GND)
- net RAND: now also U3.4
- net SP0: now also U1.3 (QA)
- net SP1: now also U70.2; no longer U1.3 (QA)
- net SP2: no longer U70.2
- net SP_RAND: now also U3.1
- net ZL_RAND: now also U3.2
