File: fulladder.kicad_sch (KiCad schematic)
At the start: 5 parts, among them U44 74AHC1G86, U45 74AHC1G08, U46 74AHC1G08, U47 74AHC1G86, U48 74AHC1G32

Commit message: very big comit what i did is in the description
jooo so this is what i did i fixed all erc errors now it is basicly finished and also started to make a website where you can lern how this whole thing works and also have a simulation for it but it is still in progress so right now chapter 1 is complete with all the simulations and right now i am working on chapter 6 it should not take very long untill i am finished i will probaply post more comits in the future so yea sry that i forgot to do that ig
Connections:
- net +3V3: now also U48.5 (VCC)
- net at U44.4, U47.1: now also U46.1
Changed lines of the file:
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@@
+	)
+	(junction
+		(at 128.27 54.61)
+		(diameter 0)
+		(color 0 0 0 0)
 	)
 	(junction
@@
 	(wire
 		(pts
-			(xy 123.19 54.61) (xy 123.19 97.79)
-		)
-		(stroke
-			(width 0)
-			(type default)
-		)
-	)
-	(wire
-		(pts
 			(xy 87.63 57.15) (xy 92.71 57.15)
 		)
@@
 	(wire
 		(pts
+			(xy 128.27 95.25) (xy 124.46 95.25)
+		)
+		(stroke
+			(width 0)
+			(type default)
+		)
+	)
+	(wire
+		(pts
 			(xy 133.35 54.61) (xy 133.35 60.96)
 		)
@@
 	(wire
 		(pts
+			(xy 124.46 95.25) (xy 124.46 97.79)
+		)
+		(stroke
+			(width 0)
+			(type default)
+		)
+	)
+	(wire
+		(pts
 			(xy 87.63 52.07) (xy 96.52 52.07)
 		)
@@
 	(wire
 		(pts
+			(xy 128.27 54.61) (xy 128.27 95.25)
+		)
+		(stroke
+			(width 0)
+			(type default)
+		)
+	)
+	(wire
+		(pts
 			(xy 92.71 57.15) (xy 92.71 78.74)
 		)
@@
 	(wire
 		(pts
-			(xy 123.19 97.79) (xy 124.46 97.79)
-		)
-		(stroke
-			(width 0)
-			(type default)
-		)
-	)
-	(wire
-		(pts
 			(xy 132.08 71.12) (xy 133.35 66.04)
 		)
@@
 	(wire
 		(pts
+			(xy 128.27 54.61) (xy 133.35 54.61)
+		)
+		(stroke
+			(width 0)
+			(type default)
+		)
+	)
+	(wire
+		(pts
 			(xy 92.71 78.74) (xy 96.52 78.74)
 		)
@@
 	(wire
 		(pts
-			(xy 125.73 54.61) (xy 133.35 54.61)
+			(xy 125.73 54.61) (xy 128.27 54.61)
 		)
 		(stroke
@@
 	(symbol
 		(lib_id "power:+3V3")
+		(at 167.64 87.63 0)
+		(unit 1)
+		(body_style 1)
+		(exclude_from_sim no)
+		(in_bom yes)
+		(on_board yes)
+		(in_pos_files yes)
+		(dnp no)
+		(fields_autoplaced yes)
+		(property "Reference" "#PWR0180"
+			(at 167.64 91.44 0)
+			(hide yes)
+			(show_name no)
+			(do_not_autoplace no)
+			(effects
+				(font
+					(size 1.27 1.27)
+				)
+			)
+		)
+		(property "Value" "+3V3"
+			(at 167.64 82.55 0)
+			(show_name no)
+			(do_not_autoplace no)
+			(effects
+				(font
+					(size 1.27 1.27)
+				)
+			)
+		)
+		(property "Footprint" "Package_DFN_QFN:Diodes_UDFN3810-9_TYPE_B"
+			(at 167.64 87.63 0)
+			(hide yes)
+			(show_name no)
+			(do_not_autoplace no)
+			(effects
+				(font
+					(size 1.27 1.27)
+				)
+			)
+		)
+		(property "Datasheet" ""
+			(at 167.64 87.63 0)
+			(hide yes)
+			(show_name no)
+			(do_not_autoplace no)
+			(effects
+				(font
+					(size 1.27 1.27)
+				)
+			)
+		)
+		(property "Description" "Power symbol creates a global label with name \"+3V3\""
+			(at 167.64 87.63 0)
+			(hide yes)
+			(show_name no)
+			(do_not_autoplace no)
+			(effects
+				(font
+					(size 1.27 1.27)
+				)
+			)
+		)
+		(pin "1"
+		)
+		(instances
+			(project "game_of_logicgatess"
+				(path "/971c6b5a-836c-4d36-bf8c-da49bad67e6d/aa8a5c47-fc35-4c5a-8837-8731560a8575/431affb0-147a-4519-9b8e-15360a5af8cd"
+					(reference "#PWR0183")
+					(unit 1)
+				)
+				(path "/971c6b5a-836c-4d36-bf8c-da49bad67e6d/aa8a5c47-fc35-4c5a-8837-8731560a8575/7879aaf0-3940-4eeb-b277-7ff442f6b7a8"
+					(reference "#PWR0180")
+					(unit 1)
+				)
+				(path "/971c6b5a-836c-4d36-bf8c-da49bad67e6d/aa8a5c47-fc35-4c5a-8837-8731560a8575/8a2b2a92-605a-4779-8962-a968838a0027"
+					(reference "#PWR0181")
+					(unit 1)
+				)
+				(path "/971c6b5a-836c-4d36-bf8c-da49bad67e6d/aa8a5c47-fc35-4c5a-8837-8731560a8575/e780d2e5-09a7-412c-ad65-7441ad6db931"
+					(reference "#PWR0182")
+					(unit 1)
+				)
+			)
+		)
+	)
+	(symbol
+		(lib_id "power:+3V3")
 		(at 148.59 53.34 0)
 		(unit 1)
@@
 					(unit 1)
 				)
-			)
-		)
-	)
-	(symbol
-		(lib_id "power:PWR_FLAG")
-		(at 167.64 87.63 0)
-		(unit 1)
-		(body_style 1)
-		(exclude_from_sim no)
-		(in_bom yes)
-		(on_board yes)
-		(in_pos_files yes)
-		(dnp no)
-		(fields_autoplaced yes)
-		(property "Reference" "#FLG04"
-			(at 167.64 85.725 0)
-			(hide yes)
-			(show_name no)
-			(do_not_autoplace no)
-			(effects
-				(font
-					(size 1.27 1.27)
-				)
-			)
-		)
-		(property "Value" "PWR_FLAG"
-			(at 167.64 82.55 0)
-			(show_name no)
-			(do_not_autoplace no)
-			(effects
-				(font
-					(size 1.27 1.27)
-				)
-			)
-		)
-		(property "Footprint" "Package_SO:TSSOP-28_4.4x9.7mm_P0.65mm"
-			(at 167.64 87.63 0)
-			(hide yes)
-			(show_name no)
-			(do_not_autoplace no)
-			(effects
-				(font
-					(size 1.27 1.27)
-				)
-			)
-		)
-		(property "Datasheet" ""
-			(at 167.64 87.63 0)
-			(hide yes)
-			(show_name no)
-			(do_not_autoplace no)
-			(effects
-				(font
-					(size 1.27 1.27)
-				)
-			)
-		)
-		(property "Description" "Special symbol for telling ERC where power comes from"
-			(at 167.64 87.63 0)
-			(hide yes)
-			(show_name no)
-			(do_not_autoplace no)
-			(effects
-				(font
-					(size 1.27 1.27)
-				)
-			)
-		)
-		(pin "1"
-		)
-		(instances
-			(project "game_of_logicgatess"
-				(path "/971c6b5a-836c-4d36-bf8c-da49bad67e6d/aa8a5c47-fc35-4c5a-8837-8731560a8575/431affb0-147a-4519-9b8e-15360a5af8cd"
-					(reference "#FLG07")
-					(unit 1)
-				)
-				(path "/971c6b5a-836c-4d36-bf8c-da49bad67e6d/aa8a5c47-fc35-4c5a-8837-8731560a8575/7879aaf0-3940-4eeb-b277-7ff442f6b7a8"
-					(reference "#FLG04")
-					(unit 1)
-				)
-				(path "/971c6b5a-836c-4d36-bf8c-da49bad67e6d/aa8a5c47-fc35-4c5a-8837-8731560a8575/8a2b2a92-605a-4779-8962-a968838a0027"
-					(reference "#FLG05")
-					(unit 1)
-				)
-				(path "/971c6b5a-836c-4d36-bf8c-da49bad67e6d/aa8a5c47-fc35-4c5a-8837-8731560a8575/e780d2e5-09a7-412c-ad65-7441ad6db931"
-					(reference "#FLG06")
-					(unit 1)
-				)
