File: mux.kicad_sch (KiCad schematic)
At the start: 8 parts, among them SW71 SW_Push, U26 74HC74, U27 74AHC1G02, U28 74AHC1G08, U29 74AHC1G08, U30 74AHC1G32

Commit message: very big comit what i did is in the description
jooo so this is what i did i fixed all erc errors now it is basicly finished and also started to make a website where you can lern how this whole thing works and also have a simulation for it but it is still in progress so right now chapter 1 is complete with all the simulations and right now i am working on chapter 6 it should not take very long untill i am finished i will probaply post more comits in the future so yea sry that i forgot to do that ig
Parts:
- added unit 3 of U26
Connections:
- net +3V3: now also U26.14 (VCC)
- net GND: now also U26.7 (GND)
