File: ring.kicad_sch (KiCad schematic)
At the start: 28 parts, among them U12 74AHC273, U13 74AHC273, U14 74AHC273, U15 74AHC273, U16 74AHC273, U17 74AHC273, U18 74AHC273, U19 74AHC273, U20 74AHC273, U21 74AHC273, U22 74AHC273, U23 74AHC273, U24 74AHC273, U25 74AHC273

Commit message: very big comit what i did is in the description
jooo so this is what i did i fixed all erc errors now it is basicly finished and also started to make a website where you can lern how this whole thing works and also have a simulation for it but it is still in progress so right now chapter 1 is complete with all the simulations and right now i am working on chapter 6 it should not take very long untill i am finished i will probaply post more comits in the future so yea sry that i forgot to do that ig
Connections:
- net CLEAR_N: now also U14.1 (~{Mr}), U19.1 (~{Mr}), U24.1 (~{Mr})
- net GND: now also C9.2, U21.10 (GND)
- net No-Context-X: no longer names the net of U25.19 (Q7)
- no-connect marks 0 -> 1
