File: untitled.kicad_sch (KiCad schematic)
At the start: 4 parts, among them U40 74AHC1G02, U41 74AHC1G32, U42 74AHC1G08, U43 74AHC1G08

Commit message: very big comit what i did is in the description
jooo so this is what i did i fixed all erc errors now it is basicly finished and also started to make a website where you can lern how this whole thing works and also have a simulation for it but it is still in progress so right now chapter 1 is complete with all the simulations and right now i am working on chapter 6 it should not take very long untill i am finished i will probaply post more comits in the future so yea sry that i forgot to do that ig
Connections:
- net VCC is gone; now on net +3V3: U41.5 (VCC), U42.5 (VCC), U43.5 (VCC)
- net +3V3: now reaches U40.5 (VCC)
